File: compaq-mx-11800.kicad_pcb (KiCad board)
At the start: 2 copper layers, 389.5 x 166.4 mm, 240 parts, among them J1 Conn_01x16_Female, J2 Conn_01x16_Female

Commit message: reorder col and row pins
Parts:
- MX74: footprint MX_Only:MXOnly-ISO-ROTATED-ReversedStabilizers-NoLED -> MX_Only:MXOnly-ISO-ReversedStabilizers-NoLED
Connections:
- D1 pad 1: row14 -> row6
- D10 pad 1: row14 -> row6
- D100 pad 1: row3 -> row11
- D101 pad 1: row2 -> row10
- D102 pad 1: row3 -> row11
- D103 pad 1: row2 -> row10
- D104 pad 1: row3 -> row11
- D105 pad 1: row2 -> row10
- D107 pad 1: row3 -> row11
- D108 pad 1: row0 -> row13
- D11 pad 1: row13 -> row4
- D114 pad 1: row0 -> row13
- D115 pad 1: row1 -> row12
- D116 pad 1: row1 -> row12
- D117 pad 1: row0 -> row13
- D118 pad 1: row1 -> row12
- D12 pad 1: row14 -> row6
- D120 pad 1: row0 -> row13
- D121 pad 1: row0 -> row13
- D122 pad 1: row1 -> row12
- D124 pad 1: row0 -> row13
- D13 pad 1: row14 -> row6
- D14 pad 1: row13 -> row4
- D15 pad 1: row14 -> row6
- D16 pad 1: row13 -> row4
- D18 pad 1: row12 -> row7
- D19 pad 1: row11 -> row5
- D2 pad 1: row14 -> row6
- D20 pad 1: row12 -> row7
- D21 pad 1: row11 -> row5
- D22 pad 1: row12 -> row7
- D23 pad 1: row11 -> row5
- D24 pad 1: row12 -> row7
- D25 pad 1: row11 -> row5
- D26 pad 1: row12 -> row7
- D27 pad 1: row12 -> row7
- D28 pad 1: row12 -> row7
- D29 pad 1: row11 -> row5
- D3 pad 1: row13 -> row4
- D30 pad 1: row12 -> row7
- D31 pad 1: row10 -> row3
- D32 pad 1: row11 -> row5
- D33 pad 1: row7 -> row0
- D34 pad 1: row9 -> row2
- D35 pad 1: row10 -> row3
- D36 pad 1: row8 -> row1
- D37 pad 1: row9 -> row2
- D38 pad 1: row10 -> row3
- D39 pad 1: row9 -> row2
- D4 pad 1: row14 -> row6
- D40 pad 1: row10 -> row3
- D41 pad 1: row9 -> row2
- D42 pad 1: row10 -> row3
- D43 pad 1: row9 -> row2
- D44 pad 1: row10 -> row3
- D45 pad 1: row9 -> row2
- D46 pad 1: row10 -> row3
- D47 pad 1: row9 -> row2
- D48 pad 1: row10 -> row3
- D49 pad 1: row9 -> row2
- D5 pad 1: row13 -> row4
- D51 pad 1: row9 -> row2
- D53 pad 1: row3 -> row11
- D54 pad 1: row5 -> row9
- D55 pad 1: row6 -> row8
- D56 pad 1: row2 -> row10
- D57 pad 1: row3 -> row11
- D58 pad 1: row7 -> row0
- D59 pad 1: row8 -> row1
- D6 pad 1: row14 -> row6
- D60 pad 1: row7 -> row0
- D61 pad 1: row8 -> row1
- D62 pad 1: row7 -> row0
- D63 pad 1: row8 -> row1
- D64 pad 1: row7 -> row0
- D65 pad 1: row8 -> row1
- D66 pad 1: row7 -> row0
- D67 pad 1: row8 -> row1
- D68 pad 1: row7 -> row0
- D69 pad 1: row8 -> row1
- D7 pad 1: row13 -> row4
- D70 pad 1: row7 -> row0
- D71 pad 1: row8 -> row1
- D72 pad 1: row1 -> row12
- D73 pad 1: row2 -> row10
- D74 pad 1: row6 -> row8
- D76 pad 1: row5 -> row9
- D77 pad 1: row6 -> row8
- D78 pad 1: row5 -> row9
- D79 pad 1: row6 -> row8
- D8 pad 1: row14 -> row6
- D80 pad 1: row5 -> row9
- D81 pad 1: row6 -> row8
- D82 pad 1: row5 -> row9
- D83 pad 1: row6 -> row8
- D84 pad 1: row5 -> row9
- D85 pad 1: row6 -> row8
- D86 pad 1: row5 -> row9
- D87 pad 1: row6 -> row8
- D88 pad 1: row5 -> row9
- D9 pad 1: row13 -> row4
- D91 pad 1: row0 -> row13
- D92 pad 1: row3 -> row11
- D94 pad 1: row3 -> row11
- D95 pad 1: row2 -> row10
- D96 pad 1: row3 -> row11
- D97 pad 1: row2 -> row10
- D98 pad 1: row3 -> row11
- D99 pad 1: row2 -> row10
- J1 pad 11: row6 -> row8
- J1 pad 12: row5 -> row9
- J1 pad 13: row2 -> row10
- J1 pad 14: row3 -> row11
- J1 pad 15: row1 -> row12
- J1 pad 16: row0 -> row13
- J1 pad 2: row7 -> row0
- J1 pad 3: row8 -> row1
- J1 pad 4: row9 -> row2
- J1 pad 5: row10 -> row3
- J1 pad 6: row13 -> row4
- J1 pad 7: row11 -> row5
- J1 pad 8: row14 -> row6
- J1 pad 9: row12 -> row7
- J2 pad 10: Net-(J2-Pad10) -> col8
- J2 pad 11: Net-(J2-Pad11) -> col9
- J2 pad 2: Net-(J2-Pad2) -> col0
- J2 pad 3: Net-(J2-Pad3) -> col1
- J2 pad 4: Net-(J2-Pad4) -> col2
- J2 pad 5: Net-(J2-Pad5) -> col3
- J2 pad 6: Net-(J2-Pad6) -> col4
- J2 pad 7: Net-(J2-Pad7) -> col5
- J2 pad 8: Net-(J2-Pad8) -> col6
- J2 pad 9: Net-(J2-Pad9) -> col7
- MX1 pad 1: col0 -> col3
- MX10 pad 1: Net-(MX10-Pad1) -> col5
- MX100 pad 1: Net-(MX100-Pad1) -> col0
- MX101 pad 1: Net-(MX100-Pad1) -> col0
- MX102 pad 1: Net-(MX102-Pad1) -> col4
- MX103 pad 1: Net-(MX102-Pad1) -> col4
- MX104 pad 1: Net-(MX10-Pad1) -> col5
- MX105 pad 1: Net-(MX10-Pad1) -> col5
- MX106 pad 1: Net-(MX106-Pad1) -> col6
- MX107 pad 1: Net-(MX106-Pad1) -> col6
- MX108 pad 1: Net-(MX108-Pad1) -> col7
- MX109 pad 1: Net-(MX10-Pad1) -> col5
- MX11 pad 1: Net-(MX106-Pad1) -> col6
- MX110 pad 1: Net-(MX10-Pad1) -> col5
- MX111 pad 1: col0 -> col3
- MX112 pad 1: col0 -> col3
- MX113 pad 1: Net-(MX100-Pad1) -> col0
- MX114 pad 1: Net-(MX114-Pad1) -> col9
- MX115 pad 1: Net-(MX114-Pad1) -> col9
- MX116 pad 1: Net-(MX108-Pad1) -> col7
- MX117 pad 1: Net-(MX10-Pad1) -> col5
- MX118 pad 1: Net-(MX10-Pad1) -> col5
- MX119 pad 1: Net-(MX106-Pad1) -> col6
- MX12 pad 1: Net-(MX106-Pad1) -> col6
- MX120 pad 1: Net-(MX100-Pad1) -> col0
- MX121 pad 1: col0 -> col3
- MX122 pad 1: col0 -> col3
- MX124 pad 1: Net-(MX106-Pad1) -> col6
- MX17 pad 1: Net-(MX17-Pad1) -> col8
- MX18 pad 1: Net-(MX18-Pad1) -> col2
- MX19 pad 1: Net-(MX18-Pad1) -> col2
- MX2 pad 1: Net-(MX18-Pad1) -> col2
- MX20 pad 1: Net-(MX20-Pad1) -> col1
- MX21 pad 1: Net-(MX20-Pad1) -> col1
- MX22 pad 1: Net-(MX100-Pad1) -> col0
- MX23 pad 1: Net-(MX100-Pad1) -> col0
- MX24 pad 1: Net-(MX102-Pad1) -> col4
- MX25 pad 1: Net-(MX10-Pad1) -> col5
- MX26 pad 1: Net-(MX10-Pad1) -> col5
- MX27 pad 1: Net-(MX106-Pad1) -> col6
- MX3 pad 1: Net-(MX18-Pad1) -> col2
- MX31 pad 1: Net-(MX106-Pad1) -> col6
- MX33 pad 1: Net-(MX17-Pad1) -> col8
- MX37 pad 1: col0 -> col3
- MX38 pad 1: col0 -> col3
- MX39 pad 1: Net-(MX18-Pad1) -> col2
- MX4 pad 1: Net-(MX20-Pad1) -> col1
- MX40 pad 1: Net-(MX18-Pad1) -> col2
- MX41 pad 1: Net-(MX20-Pad1) -> col1
- MX42 pad 1: Net-(MX20-Pad1) -> col1
- MX43 pad 1: Net-(MX100-Pad1) -> col0
- MX44 pad 1: Net-(MX100-Pad1) -> col0
- MX45 pad 1: Net-(MX102-Pad1) -> col4
- MX46 pad 1: Net-(MX102-Pad1) -> col4
- MX47 pad 1: Net-(MX10-Pad1) -> col5
- MX48 pad 1: Net-(MX10-Pad1) -> col5
- MX49 pad 1: Net-(MX106-Pad1) -> col6
- MX5 pad 1: Net-(MX20-Pad1) -> col1
- MX50 pad 1: Net-(MX106-Pad1) -> col6
- MX51 pad 1: Net-(MX108-Pad1) -> col7
- MX52 pad 1: Net-(MX17-Pad1) -> col8
- MX57 pad 1: Net-(MX114-Pad1) -> col9
- MX58 pad 1: col0 -> col3
- MX59 pad 1: col0 -> col3
- MX6 pad 1: Net-(MX100-Pad1) -> col0
- MX60 pad 1: Net-(MX18-Pad1) -> col2
- MX61 pad 1: Net-(MX18-Pad1) -> col2
- MX62 pad 1: Net-(MX20-Pad1) -> col1
- MX63 pad 1: Net-(MX20-Pad1) -> col1
- MX64 pad 1: Net-(MX100-Pad1) -> col0
- MX65 pad 1: Net-(MX100-Pad1) -> col0
- MX66 pad 1: Net-(MX102-Pad1) -> col4
- MX67 pad 1: Net-(MX102-Pad1) -> col4
- MX68 pad 1: Net-(MX10-Pad1) -> col5
- MX69 pad 1: Net-(MX10-Pad1) -> col5
- MX7 pad 1: Net-(MX100-Pad1) -> col0
- MX70 pad 1: Net-(MX106-Pad1) -> col6
- MX71 pad 1: Net-(MX108-Pad1) -> col7
- MX74 pad 1: Net-(MX108-Pad1) -> col7
- MX75 pad 1: col0 -> col3
- MX76 pad 1: col0 -> col3
- MX77 pad 1: col0 -> col3
- MX78 pad 1: Net-(MX18-Pad1) -> col2
- MX79 pad 1: Net-(MX18-Pad1) -> col2
- MX8 pad 1: Net-(MX102-Pad1) -> col4
- MX80 pad 1: Net-(MX20-Pad1) -> col1
- MX81 pad 1: Net-(MX20-Pad1) -> col1
- MX82 pad 1: Net-(MX100-Pad1) -> col0
- MX83 pad 1: Net-(MX100-Pad1) -> col0
- MX84 pad 1: Net-(MX102-Pad1) -> col4
- MX85 pad 1: Net-(MX102-Pad1) -> col4
- MX86 pad 1: Net-(MX10-Pad1) -> col5
- MX87 pad 1: Net-(MX10-Pad1) -> col5
- MX88 pad 1: Net-(MX106-Pad1) -> col6
- MX89 pad 1: Net-(MX108-Pad1) -> col7
- MX9 pad 1: Net-(MX10-Pad1) -> col5
- MX90 pad 1: Net-(MX17-Pad1) -> col8
- MX91 pad 1: Net-(MX17-Pad1) -> col8
- MX92 pad 1: Net-(MX108-Pad1) -> col7
- MX93 pad 1: col0 -> col3
- MX94 pad 1: col0 -> col3
- MX95 pad 1: col0 -> col3
- MX96 pad 1: Net-(MX18-Pad1) -> col2
- MX97 pad 1: Net-(MX18-Pad1) -> col2
- MX98 pad 1: Net-(MX20-Pad1) -> col1
- MX99 pad 1: Net-(MX20-Pad1) -> col1
- MX_*1 pad 1: Net-(MX17-Pad1) -> col8
- MX_-1 pad 1: Net-(MX17-Pad1) -> col8
- MX_/1 pad 1: Net-(MX108-Pad1) -> col7
- MX_7 pad 1: Net-(MX108-Pad1) -> col7
- MX_P+1 pad 1: Net-(MX17-Pad1) -> col8
- MX_P,1 pad 1: Net-(MX114-Pad1) -> col9
- MX_P0 pad 1: Net-(MX17-Pad1) -> col8
- MX_P1 pad 1: Net-(MX17-Pad1) -> col8
- MX_P2 pad 1: Net-(MX17-Pad1) -> col8
- MX_P3 pad 1: Net-(MX17-Pad1) -> col8
- MX_P4 pad 1: Net-(MX17-Pad1) -> col8
- MX_P5 pad 1: Net-(MX17-Pad1) -> col8
- MX_P6 pad 1: Net-(MX17-Pad1) -> col8
- MX_P8 pad 1: Net-(MX108-Pad1) -> col7
- MX_P9 pad 1: Net-(MX17-Pad1) -> col8
- MX_Penter1 pad 1: Net-(MX17-Pad1) -> col8
- MX_numlock1 pad 1: Net-(MX108-Pad1) -> col7
Routing:
- net col3: track 0.00 -> 912.3 mm
- net col2: track 0.00 -> 768.8 mm
- net Net-(MX18-Pad1): track 767.5 -> 0.00 mm
- net col1: track 0.00 -> 643.8 mm
- net Net-(MX20-Pad1): track 642.5 -> 0.00 mm
- net Net-(MX100-Pad1): track 601.7 -> 0.00 mm
- net col9: track 0.00 -> 573.5 mm
- net col8: track 0.00 -> 569.9 mm
- net Net-(MX114-Pad1): track 520.0 -> 0.00 mm
- net Net-(MX17-Pad1): track 518.6 -> 0.00 mm
- net row13: track 356.2 -> 835.7 mm
- net col7: track 0.00 -> 478.1 mm
- net Net-(MX108-Pad1): track 462.1 -> 0.00 mm
- net row4: track 0.00 -> 448.9 mm
- net col5: track 0.00 -> 443.4 mm
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
Commit message: add filled zones
Parts:
- MX1, MX10, MX11, MX12, MX17, MX18, MX19, MX2, MX20, MX21, MX22, MX23, MX24, MX25, MX26, MX27, MX3, MX4, MX5, MX6, MX7, MX8, MX9: footprint MX_Only:MXOnly-1U-NoLED -> MX_Alps_Hybrid:MX-1U-NoLED
Connections:
- net Net-(J1-Pad1) renamed GND
Routing:
- added copper zone on F.Cu, net (none)
