File: va11800.kicad_pcb (KiCad board)
At the start: 2 copper layers, 389.5 x 166.4 mm, 256 parts, among them J1 Conn_01x16_Female, J2 Conn_01x16_Female, j1 MX-NoLED, k1 MX-NoLED, m1 MX-NoLED, p1 MX-NoLED, q1 MX-NoLED, t1 MX-NoLED, u1 MX-NoLED, x1 MX-NoLED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

Commit message: modify GND pad
Parts:
- removed H6, H7: MountingHole_Pad, Keebio-Parts:SolidCopper
- added J6: D2, Keebio-Parts:SinglePad, F.Cu at (258.2, 62.3)
- added J6: D2, Keebio-Parts:SinglePad, F.Cu at (392.0, 162.9)
Routing:
- net GND: track 508.1 -> 511.4 mm, vias 2 -> 4
